Commit message: real scene

File: models/dinnerware/pan_tefal.urdf (robot description, URDF)
Before this commit: robot cube, 1 links, 0 joints
Links:
- link cube: mass 2. -> 0.001

File: models/drake/objects/gripper.urdf (robot description, URDF)
Before this commit: robot cube_gripper, 8 links, 7 joints
Joints:
- joint txj: limit lower=-0.5 upper=0.5 -> lower=-1.0 upper=1.0
- joint tyj: limit lower=-0.5 upper=0.5 -> lower=-1.0 upper=1.0
- joint tzj: limit lower=-1.5 upper=0.5 -> lower=0 upper=2.0
